File: LPC5514-USB-Extend.kicad_pcb (KiCad board)
At the start: 2 copper layers, 55 parts, among them J1 USB_C_Receptacle_USB2.0, J2 Conn_02x05_Odd_Even, J3 Conn_02x08_Counter_Clockwise, J4 Conn_01x04, J5 Conn_02x05_Odd_Even, J6 Screw_Terminal_01x03, J7 Conn_02x10_Odd_Even, U1 LPC5514JBD64E, U2 AP1117-33, U3 TJA1042T-3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

Commit message: update pcb
Parts:
- C1, C12, C14, C15, C17, C18, C19, C2, C22, C25, C26, C8, R8, R9: moved to B.Cu
- L1: footprint Resistor_SMD:R_0603_1608Metric -> Inductor_SMD:L_Wuerth_MAPI-2512
- R1: value 5K1 -> DNP; moved to B.Cu
- R2: value DNP -> 5K1; moved to B.Cu
- moved D2 78.8 mm to (103.2, 113.9), turned to 180 degrees
- moved R5 78.8 mm to (106.7, 111.9)
- moved C7 74.0 mm to (105.2, 90.6), turned to 180 degrees
- moved C4 73.9 mm to (102.6, 92.8), turned to 180 degrees
- moved J1 73.2 mm to (96.3, 101.5), turned to 270 degrees
- moved R2 71.1 mm to (103.2, 100.7), turned to 180 degrees
- moved C9 70.2 mm to (105.8, 93.7), turned to 270 degrees
- moved FB1 69.4 mm to (103.0, 94.7), turned to 180 degrees
- moved D3 69.0 mm to (103.2, 111.9), turned to 180 degrees
- moved C14 68.1 mm to (114.8, 96.3), turned to 90 degrees
- moved R4 65.5 mm to (106.7, 113.8)
- moved L1 63.4 mm to (116.5, 109.3), turned to 270 degrees
- moved C5 61.1 mm to (114.6, 106.7)
- moved R1 60.1 mm to (103.2, 102.3), turned to 180 degrees
- moved C25 58.2 mm to (125.5, 99.3), turned to 270 degrees
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Connections:
- net /USB_DM renamed Net-(J1-PadB7)
- net /USB_DP renamed Net-(J1-PadB6)
- C7 pad 1: Net-(C7-Pad1) -> +5V
- FB2 pad 2: Net-(FB2-Pad2) -> +3V3
- J1 pad A6: Net-(J1-PadA6) -> /USB1_DP
- J1 pad A7: Net-(J1-PadA7) -> /USB1_DM
- J6 pad 1: /CANH -> /CANL
- J6 pad 3: /CANL -> /CANH
Routing:
- net /TARGET_RESET: track 0.00 -> 23.7 mm
- net /TARGET_SWO: track 0.00 -> 21.7 mm
- net /USB1_DP: track 0.00 -> 19.0 mm
- net /USB1_DM: track 0.00 -> 19.0 mm
- net /CAN0_TD: track 0.00 -> 18.2 mm
- net /TARGET_VCC: track 0.00 -> 17.7 mm
- net /CAN0_RD: track 0.00 -> 16.8 mm
- net /TARGET_SWCLK: track 0.00 -> 16.1 mm
- net /CANH: track 0.00 -> 14.3 mm
- net /TARGET_SWDIO: track 0.00 -> 14.0 mm
- net /CANL: track 0.00 -> 12.5 mm
- net /MCU_RESET: track 0.00 -> 12.0 mm, vias 0 -> 1
- net Net-(C5-Pad2): track 0.00 -> 11.3 mm
- net +5V: track 0.00 -> 10.5 mm
- net +5VA: track 0.00 -> 9.01 mm
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Other:
- net class Default: clearance 0.2 -> 0.1524; trace_width 0.25 -> 0.2032
- net class PWR added: clearance 0.1524, trace_width 0.2032, via_dia 0.8, via_drill 0.4
- rule trace_clearance: 0.2 -> 0.1524

Commit message: update design
Parts:
- added DNP1: Ferrite_Bead_Small, Inductor_SMD:L_0603_1608Metric, F.Cu at (114.3, 105.0)
- added R12: 10K, Resistor_SMD:R_0603_1608Metric, F.Cu at (133.9, 107.7)
- added R13: 20K, Resistor_SMD:R_0603_1608Metric, F.Cu at (133.9, 109.3)
- added TP1: TestPoint, TestPoint:TestPoint_Pad_1.0x1.0mm, F.Cu at (134.6, 98.2)
- added TP2: TestPoint, TestPoint:TestPoint_Pad_1.0x1.0mm, F.Cu at (134.6, 100.3)
- C17: moved to F.Cu
- moved C11 11.3 mm to (116.3, 114.3), turned to 180 degrees
- moved C17 7.51 mm to (125.3, 95.4)
- moved C21 6.76 mm to (116.1, 112.5), turned to 180 degrees
- moved C24 6.40 mm to (134.2, 102.3)
- moved C18 4.10 mm to (124.3, 95.3), turned to 90 degrees
- moved D1 3.91 mm to (103.2, 113.9)
- moved R3 3.91 mm to (106.7, 113.8)
- moved D2 3.86 mm to (103.2, 110.0)
- moved R4 3.86 mm to (106.7, 110.0), turned to 180 degrees
- moved FB1 1.76 mm to (104.7, 94.9)
- moved C4 1.74 mm to (104.3, 93.0)
- moved C9 1.68 mm to (107.5, 93.7)
- turned R5 to 180 degrees
Connections:
- D3 pad 2: Net-(D3-Pad2) -> +3V3
- J3 pad 2: /FC3_RTS_SCL_SSEL1 -> /FC3_CTS_SDA_SSEL0
- J3 pad 3: /FC3_CTS_SDA_SSEL0 -> /FC3_RTS_SCL_SSEL1
- U1 pad 57: Net-(U1-Pad57) -> /CAN_STB
Routing:
- net +3V3: track 3.57 -> 157.2 mm, vias 0 -> 10
- net GND: track 0.00 -> 111.4 mm, vias 0 -> 52
- net +5V: track 10.5 -> 86.0 mm, vias 0 -> 4
- net /TARGET_VCC_DIV: track 1.57 -> 60.6 mm, vias 0 -> 4
- net /FC3_SCK: track 0.00 -> 35.3 mm, vias 0 -> 2
- net /FC3_TXD_SCL_MISO: track 0.00 -> 28.9 mm, vias 0 -> 2
- net /LED_R: track 0.00 -> 24.0 mm
- net /LED_B: track 0.00 -> 24.0 mm
- net /CAN_STB: track 0.00 -> 23.7 mm
- net /FC3_RXD_SDA_MOSI: track 0.00 -> 22.3 mm, vias 0 -> 2
- net Net-(J1-PadS1): track 0.00 -> 21.3 mm
- net +5VA: track 9.01 -> 28.4 mm
- net /LED_G: track 6.40 -> 23.9 mm
- net /FC3_RTS_SCL_SSEL1: track 0.00 -> 15.2 mm
- net /FC3_CTS_SDA_SSEL0: track 0.00 -> 13.3 mm
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- added copper zone on F.Cu, net +3V3
- added copper zone on F.Cu, net +5V
- added copper zone on F.Cu, net +5VA
- added copper zone on B.Cu, net GND
Other:
- board outline added: 81 x 31 mm

Commit message: update pcb & add data manual
Parts:
- J1: footprint Connector_USB:USB_C_Receptacle_Amphenol_12401548E4-2A -> Connector_USB:USB_C_Receptacle_HRO_TYPE-C-31-M-12
- moved J1 0.17 mm to (96.1, 101.5)
Routing:
- net Net-(J1-PadS1): track 21.3 -> 1.42 mm
- net +5VA: track 28.4 -> 39.6 mm
- net Net-(J1-PadB5): track 12.5 -> 3.65 mm, vias 0 -> 1
- net /USB1_DP: track 19.0 -> 22.0 mm
- net /USB1_DM: track 19.0 -> 21.5 mm
- net GND: track 111.4 -> 110.1 mm, vias 52 -> 53
- net Net-(J1-PadA5): track 2.78 -> 3.68 mm
